File: electronics/crt-driver.sch (KiCad schematic (older format))
At the start: 10 parts

Commit message: Design notes for 3.3V LDR and schematic updates
Connections:
- net GNDD is gone; now on net GND: R?.2
- net +6V renamed +5V
- net GND1 renamed GND
Changed lines of the file:
@@
 $EndComp
 $Comp
-L power:GND1 #PWR?
+L power:GND #PWR?
 U 1 1 6115E955
 P 9000 2150
@@
 AR Path="/6113F6B3/6115E955" Ref="#PWR?"  Part="1"
 F 0 "#PWR?" H 9000 1900 50  0001 C CNN
-F 1 "GND1" H 9000 2000 50  0000 C CNN
+F 1 "GND" H 9000 2000 50  0000 C CNN
 F 2 "" H 9000 2150 50  0001 C CNN
 F 3 "" H 9000 2150 50  0001 C CNN
@@
 	9000 2050 9000 2150
 $Comp
-L power:+6V #PWR?
+L power:+5V #PWR?
 U 1 1 6115E95C
 P 9000 1050
@@
 AR Path="/6113F6B3/6115E95C" Ref="#PWR?"  Part="1"
 F 0 "#PWR?" H 9000 900 50  0001 C CNN
-F 1 "+6V" H 9000 1190 50  0000 C CNN
+F 1 "+5V" H 9000 1190 50  0000 C CNN
 F 2 "" H 9000 1050 50  0001 C CNN
 F 3 "" H 9000 1050 50  0001 C CNN
@@
 	9200 950  9200 1150
 $Comp
-L power:GND1 #PWR?
+L power:GND #PWR?
 U 1 1 6115E965
 P 9300 950
@@
 AR Path="/6113F6B3/6115E965" Ref="#PWR?"  Part="1"
 F 0 "#PWR?" H 9300 700 50  0001 C CNN
-F 1 "GND1" H 9300 800 50  0000 C CNN
+F 1 "GND" H 9300 800 50  0000 C CNN
 F 2 "" H 9300 950 50  0001 C CNN
 F 3 "" H 9300 950 50  0001 C CNN
@@
 	1    0    0    -1
 $EndComp
-$Comp
-L power:GND1 #PWR?
-U 1 1 6115E983
-P 9950 3300
-AR Path="/6115E983" Ref="#PWR?"  Part="1"
-AR Path="/6113F6B3/6115E983" Ref="#PWR?"  Part="1"
-F 0 "#PWR?" H 9950 3050 50  0001 C CNN
-F 1 "GND1" H 9950 3150 50  0000 C CNN
-F 2 "" H 9950 3300 50  0001 C CNN
-F 3 "" H 9950 3300 50  0001 C CNN
-	1    9950 3300
-	1    0    0    -1
-$EndComp
 Text Notes 10150 2950 0    50   ~ 0
 Adjustable focus\nclamped between\napprox. 0V...+100V
@@
 $EndComp
 $Comp
-L power:GND1 #PWR?
+L power:GND #PWR?
 U 1 1 6115E9BA
 P 9150 4900
@@
 AR Path="/6113F6B3/6115E9BA" Ref="#PWR?"  Part="1"
 F 0 "#PWR?" H 9150 4650 50  0001 C CNN
-F 1 "GND1" H 9150 4750 50  0000 C CNN
+F 1 "GND" H 9150 4750 50  0000 C CNN
 F 2 "" H 9150 4900 50  0001 C CNN
 F 3 "" H 9150 4900 50  0001 C CNN
@@
 Connection ~ 9500 4600
 $Comp
-L power:GNDD #PWR?
+L power:GND #PWR?
 U 1 1 6115E9CF
 P 9500 4900
@@
 AR Path="/6113F6B3/6115E9CF" Ref="#PWR?"  Part="1"
 F 0 "#PWR?" H 9500 4650 50  0001 C CNN
-F 1 "GNDD" H 9500 4750 50  0000 C CNN
+F 1 "GND" H 9500 4750 50  0000 C CNN
 F 2 "" H 9500 4900 50  0001 C CNN
 F 3 "" H 9500 4900 50  0001 C CNN
@@
 CUTOFF
 $Comp
-L power:GND1 #PWR?
+L power:GND #PWR?
 U 1 1 6115E9F3
 P 9800 4900
@@
 AR Path="/6113F6B3/6115E9F3" Ref="#PWR?"  Part="1"
 F 0 "#PWR?" H 9800 4650 50  0001 C CNN
-F 1 "GND1" H 9800 4750 50  0000 C CNN
+F 1 "GND" H 9800 4750 50  0000 C CNN
 F 2 "" H 9800 4900 50  0001 C CNN
 F 3 "" H 9800 4900 50  0001 C CNN
@@
 Text HLabel 9500 4300 1    50   Input ~ 0
 ~BLANK
+$Comp
+L power:GND #PWR?
+U 1 1 6115E983
+P 9950 3300
+AR Path="/6115E983" Ref="#PWR?"  Part="1"
+AR Path="/6113F6B3/6115E983" Ref="#PWR?"  Part="1"
+F 0 "#PWR?" H 9950 3050 50  0001 C CNN
+F 1 "GND" H 9950 3150 50  0000 C CNN
+F 2 "" H 9950 3300 50  0001 C CNN
+F 3 "" H 9950 3300 50  0001 C CNN
+	1    9950 3300
+	1    0    0    -1
+$EndComp
 $EndSCHEMATC
